File: ESP32-C6FH4.kicad_pcb (KiCad board)
At the start: 4 copper layers, 40 x 25 mm, 58 parts, among them J1 USB_C_Receptacle_USB2.0_16P, J2 Micro_SD_Card, J3 CAN, J4 UART Telemetry, J5 I2C Connector, J6 External SPI Connector, SW1 SKTAAAE010, SW2 SKTAAAE010, U1 ESP32-C6FH4, U2 TC2014-3.3VxCTTR, U3 TCAN332, U4 74LVC1G125, Y1 40MHz

Commit message: add enclosure
Parts:
- added kibuzzard-6AC1ACDB: G***, kibuzzard-6AC1ACDB, B.Cu at (146.2, 66.2)
- added kibuzzard-6AC1ADD1: G***, kibuzzard-6AC1ADD1, B.Cu at (148.9, 84.3)
- added kibuzzard-6AC1ADF5: G***, kibuzzard-6AC1ADF5, B.Cu at (139.1, 84.2)
- J6: value External SPI Connector -> SPI Connector
